File: PIC18F8722_BREAKOUT_BRD.sch (KiCad schematic (older format))
At the start: 25 parts, among them IC1 PIC18F8722, P1 PGM_CONN, P12 PWR_CON, P2 CONN_16, P3 CONN_5, P4 CONN_16, P5 CONN_16, P6 CONN_16, P7 PWR_CON, P9 PWR_CON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

Commit message: Updated as per requirement
Parts:
- removed P12: PWR_CON, ~, symbol CONN_2
- removed P2, P4, P5, P6: CONN_16, ~, symbol CONN_16
- removed P3: CONN_5, ~, symbol CONN_5
- added P2: CONN _1_20, ~, symbol CONN_20
- added P3: CONN_21_40, ~, symbol CONN_20
- added P4: CONN_41_60, ~, symbol CONN_20
- added P5: CONN_61_80, ~, symbol CONN_20
Connections:
- net labels added: AVDD, AVSS, PIN11, PIN12, PIN31, PIN32, PIN48, PIN51, PIN70, PIN71, RG5
- wire segments 201 -> 210
